Commit message: Update Nav2 launch and fix URDF model

File: src/ros2_lidar/picar.urdf (robot description, URDF)
Before this commit: robot pi_car, 2 links, 1 joints
Links:
- added link base_footprint
- added link front_left_wheel_link; collision cylinder length=0.02 radius=0.0325; visual cylinder length=0.02 radius=0.0325
- added link front_right_wheel_link; collision cylinder length=0.02 radius=0.0325; visual cylinder length=0.02 radius=0.0325
- added link rear_left_wheel_link; collision cylinder length=0.02 radius=0.0325; visual cylinder length=0.02 radius=0.0325
- added link rear_right_wheel_link; collision cylinder length=0.02 radius=0.0325; visual cylinder length=0.02 radius=0.0325
- added link standoff_link; visual cylinder length=0.085 radius=0.005
- link base_link: geometry collision box size=0.14 0.18 0.09; visual box size=0.14 0.18 0.09
- link laser: geometry visual cylinder length=0.03 radius=0.035
Joints:
- added joint base_joint: type fixed, parent base_footprint, child base_link, origin xyz=0 0 50 rpy=0 0 0
- added joint front_left_wheel_joint: type continuous, parent base_link, child front_left_wheel_link, origin xyz=0.045 0.09999999999999999 -0.02 rpy=0 0 0, axis 0 1 0
- added joint front_right_wheel_joint: type continuous, parent base_link, child front_right_wheel_link, origin xyz=0.045 -0.09999999999999999 -0.02 rpy=0 0 0, axis 0 1 0
- added joint rear_left_wheel_joint: type continuous, parent base_link, child rear_left_wheel_link, origin xyz=-0.045 0.09999999999999999 -0.02 rpy=0 0 0, axis 0 1 0
- added joint rear_right_wheel_joint: type continuous, parent base_link, child rear_right_wheel_link, origin xyz=-0.045 -0.09999999999999999 -0.02 rpy=0 0 0, axis 0 1 0
- added joint standoff_joint: type fixed, parent base_link, child standoff_link, origin xyz=0.0 0 0.0875 rpy=0 0 0
- joint laser_joint: origin xyz=0 0 0.05 rpy=0 0 0 -> xyz=0.0 0 0.14500000000000002 rpy=0 0 0
