Commit message: fixed nav2

File: urdf/picar.urdf (robot description, URDF)
Before this commit: robot pi_car, 8 links, 7 joints
Joints:
- joint base_joint: origin xyz=0 0 0 rpy=0 0 0 -> xyz=0 0 0.05 rpy=0 0 0
- joint front_left_wheel_joint: origin xyz=0.045 0.09999999999999999 -0.02 rpy=0 0 0 -> xyz=0.045 0.1 -0.02 rpy=0 0 0
- joint front_right_wheel_joint: origin xyz=0.045 -0.09999999999999999 -0.02 rpy=0 0 0 -> xyz=0.045 -0.1 -0.02 rpy=0 0 0
- joint laser_joint: origin xyz=0.0 0 0.14500000000000002 rpy=0 0 0 -> xyz=0.0 0 0.145 rpy=0 0 0
- joint rear_left_wheel_joint: origin xyz=-0.045 0.09999999999999999 -0.02 rpy=0 0 0 -> xyz=-0.045 0.1 -0.02 rpy=0 0 0
- joint rear_right_wheel_joint: origin xyz=-0.045 -0.09999999999999999 -0.02 rpy=0 0 0 -> xyz=-0.045 -0.1 -0.02 rpy=0 0 0
